File: PCB/LQS-keyboard/LQS-keyboard.kicad_sch (KiCad schematic)
At the start: 65 parts, among them SW1 SW_Push, SW10 SW_Push, SW11 SW_Push, SW12 SW_Push, SW13 SW_Push, SW14 SW_Push, SW15 SW_Push, SW16 SW_Push, SW17 SW_Push, SW18 SW_Push, SW19 SW_Push, SW2 SW_Push, SW20 SW_Push, SW21 SW_Push, SW22 SW_Push, SW23 SW_Push, SW24 SW_Push, SW25 SW_Push, SW26 SW_Push, SW27 SW_Push, SW28 SW_Push, SW29 SW_Push, SW3 SW_Push, SW4 SW_Push, SW5 SW_Push, SW6 SW_Push, SW7 SW_Push, SW8 SW_Push, SW9 SW_Push, U1 XIAO-nRF52840-DIP

Commit message: 2025-07-05 update
Parts:
- removed JP3, JP4, JP5, JP6: SolderJumper_2_Open, Jumper:SolderJumper-2_P1.3mm_Open_Pad1.0x1.5mm, symbol Jumper:SolderJumper_2_Open
- removed U1: XIAO-nRF52840-DIP, seeed_xiao_ble:XIAO-nRF52840-DIP, symbol seed_xiao_ble:XIAO-nRF52840-DIP
- added D30: LED_RGBA, LED_THT:LED_D5.0mm-4_RGB, symbol Device:LED_RGBA
- added R1, R2, R3: R, Resistor_THT:R_Axial_DIN0204_L3.6mm_D1.6mm_P7.62mm_Horizontal, symbol Device:R
- added U2: ProMicro, theonepromicro:TheOneProMicro, symbol theonepromicro:ProMicro_2-Lily58-cache
- JP1, JP2: footprint Jumper:SolderJumper-2_P1.3mm_Open_Pad1.0x1.5mm -> Jumper:SolderJumper-2_P1.3mm_Open_RoundedPad1.0x1.5mm
- SW1, SW10, SW11, SW12, SW13, SW14, SW15, SW16, SW17, SW18, SW19, SW2, SW20, SW21, SW22, SW23, SW24, SW25, SW26, SW27, SW28, SW29, SW3, SW4, SW5, SW6, SW7, SW8, SW9: footprint key-switches:SW_Kailh_Choc_V1V2_THT_Hybrid -> key-switches:SW_Kailh_Choc_V1V2_THT_Hybrid_doubleside
Connections:
- net COL1: now also U2.7 (GP4)
- net COL2: now also U2.8 (GP5)
- net COL3: now also U2.9 (GP6)
- net COL4: now also U2.10 (GP7)
- net COL5: now also U2.11 (GP8)
- net COL6: now also U2.12 (GP9)
- net ROW1: now also U2.13 (GP21); no longer JP1.1 (A)
- net ROW2: now also U2.14 (GP23); no longer JP2.1 (A)
- net ROW3: now also U2.15 (GP20)
- net ROW4: now also U2.16 (GP22)
- net ROWT: now also U2.17 (GP26(A0))
- net 3v3: now reaches JP1.2 (B)
- net 3v3: now also JP2.2 (B), D30.4 (A)
- new net: JP1.1 (A), U2.4 (GND)
- new net: D30.2 (GK), R2.1
- new net: D30.1 (RK), R1.1
- new net: D30.3 (BK), R3.1
- new net: JP2.1 (A), U2.21 (3v3)
- new net LEDB: R3.2, U2.20 (GP29(A3))
- new net LEDG: R2.2, U2.19 (GP28(A2))
- new net LEDR: R1.2, U2.18 (GP27(A1))
