File: PCB/LQS-keyboard/LQS-keyboard.kicad_pcb (KiCad board)
At the start: 2 copper layers, 148.9 x 134.9 mm, 65 parts, among them SW1 SW_Push, SW10 SW_Push, SW11 SW_Push, SW12 SW_Push, SW13 SW_Push, SW14 SW_Push, SW15 SW_Push, SW16 SW_Push, SW17 SW_Push, SW18 SW_Push, SW19 SW_Push, SW2 SW_Push, SW20 SW_Push, SW21 SW_Push, SW22 SW_Push, SW23 SW_Push, SW24 SW_Push, SW25 SW_Push, SW26 SW_Push, SW27 SW_Push, SW28 SW_Push, SW29 SW_Push, SW3 SW_Push, SW4 SW_Push, SW5 SW_Push, SW6 SW_Push, SW7 SW_Push, SW8 SW_Push, SW9 SW_Push, U1 XIAO-nRF52840-DIP

Commit message: 2025-07-05 update
Parts:
- removed JP3, JP4, JP5, JP6: SolderJumper_2_Open, Jumper:SolderJumper-2_P1.3mm_Open_Pad1.0x1.5mm
- removed U1: XIAO-nRF52840-DIP, seeed_xiao_ble:XIAO-nRF52840-DIP
- added D30: LED_RGBA, LED_THT:LED_D5.0mm-4_RGB_Wide_Pins, F.Cu at (62.8, 33.6)
- added R1: R, Resistor_THT:R_Axial_DIN0204_L3.6mm_D1.6mm_P7.62mm_Horizontal, F.Cu at (75.6, 32.2)
- added R2: R, Resistor_THT:R_Axial_DIN0204_L3.6mm_D1.6mm_P7.62mm_Horizontal, F.Cu at (75.4, 29.5)
- added R3: R, Resistor_THT:R_Axial_DIN0204_L3.6mm_D1.6mm_P7.62mm_Horizontal, F.Cu at (75.4, 27.0)
- added U2: ProMicro, theonepromicro:TheOneProMicro, F.Cu at (179.1, 51.2)
- JP1, JP2: footprint Jumper:SolderJumper-2_P1.3mm_Open_Pad1.0x1.5mm -> Jumper:SolderJumper-2_P1.3mm_Open_RoundedPad1.0x1.5mm
- SW1, SW10, SW11, SW12, SW13, SW14, SW15, SW16, SW17, SW18, SW19, SW2, SW20, SW21, SW22, SW23, SW24, SW25, SW26, SW27, SW28, SW29, SW3, SW4, SW5, SW6, SW7, SW8, SW9: footprint key-switches:SW_Kailh_Choc_V1V2_THT_Hybrid -> key-switches:SW_Kailh_Choc_V1V2_THT_Hybrid_doubleside
- moved JP2 21.3 mm to (182.0, 43.6), turned to 90 degrees
- moved JP1 18.7 mm to (178.2, 43.6), turned to 90 degrees
- moved D25 1.56 mm to (172.9, 112.5)
Connections:
- JP1 pad 1: ROW1 -> Net-(JP1-A)
- JP1 pad 2: Net-(JP1-B) -> 3v3
- JP2 pad 1: ROW2 -> Net-(JP2-A)
- JP2 pad 2: Net-(JP2-B) -> 3v3
Routing:
- net 3v3: track 0.00 -> 126.8 mm
- net LEDR: track 0.00 -> 118.5 mm
- net LEDG: track 0.00 -> 116.8 mm
- net LEDB: track 0.00 -> 115.2 mm
- net COL4: track 182.1 -> 242.3 mm
- net COL6: track 98.3 -> 157.0 mm
- net COL3: track 212.0 -> 261.8 mm
- net COL5: track 167.1 -> 210.5 mm
- net Net-(JP4-A): track 36.3 -> 0.00 mm, vias 1 -> 0
- net Net-(JP5-A): track 31.1 -> 0.00 mm, vias 1 -> 0
- net COL2: track 252.7 -> 279.1 mm
- net Net-(JP6-A): track 23.3 -> 0.00 mm
- net COL1: track 221.3 -> 238.3 mm
- net Net-(JP1-B): track 15.0 -> 0.00 mm
- net Net-(D30-BK): track 0.00 -> 13.6 mm
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Other:
- outline, holes or cut-outs redrawn

Commit message: 2025-07-06 update
Parts:
- added REF**: MountingHole_2.2mm_M2, MountingHole:MountingHole_2.2mm_M2, F.Cu at (90.2, 33.8)
- added REF**: MountingHole_2.2mm_M2, MountingHole:MountingHole_2.2mm_M2, F.Cu at (182.5, 121.0)
- added REF**: MountingHole_2.2mm_M2, MountingHole:MountingHole_2.2mm_M2, F.Cu at (180.2, 58.5)
- added REF**: MountingHole_2.2mm_M2, MountingHole:MountingHole_2.2mm_M2, F.Cu at (118.5, 104.0)
Routing:
- net COL2: track 279.1 -> 279.9 mm
Other:
- board size 148.9 x 134.9 mm -> 148.9 x 134.5 mm
