File: PCB/kicad/LQS-keyboard.kicad_pcb (KiCad board)
At the start: 2 copper layers, 148.9 x 134.5 mm, 69 parts, among them SW1 SW_Push, SW10 SW_Push, SW11 SW_Push, SW12 SW_Push, SW13 SW_Push, SW14 SW_Push, SW15 SW_Push, SW16 SW_Push, SW17 SW_Push, SW18 SW_Push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

Commit message: 2025-07-07 update
Parts:
- D1, D10, D11, D12, D13, D14, D15, D16, D17, D18, D19, D2, D20, D21, D22, D23, D24, D25, D26, D27, D28, D29, D3, D4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: moved to B.Cu
